Commit message: [WIP] add dual-arm setting for UR5e

File: ur_e_description/urdf/ur5e.urdf.xacro (robot description, xacro)
@@ -82,7 +82,7 @@
           <mesh filename="package://ur_e_description/meshes/ur5e/visual/base.dae" />
         </geometry>
-        <material name="LightGrey">
-          <color rgba="0.7 0.7 0.7 1.0"/>
-        </material>
+        <!--material name="LightGrey">
+          <color rgba="0.7 0.7 0.7 1.0"/>
+        </material-->
       </visual>
       <collision>
@@ -119,7 +119,7 @@
           <mesh filename="package://ur_e_description/meshes/ur5e/visual/shoulder.dae" />
         </geometry>
-        <material name="LightGrey">
-          <color rgba="0.7 0.7 0.7 1.0"/>
-        </material>
+        <!--material name="LightGrey">
+          <color rgba="0.7 0.7 0.7 1.0"/>
+        </material-->
       </visual>
       <collision>
@@ -156,7 +156,7 @@
           <mesh filename="package://ur_e_description/meshes/ur5e/visual/upperarm.dae" />
         </geometry>
-        <material name="LightGrey">
-          <color rgba="0.7 0.7 0.7 1.0"/>
-        </material>
+        <!--material name="LightGrey">
+          <color rgba="0.7 0.7 0.7 1.0"/>
+        </material-->
       </visual>
       <collision>
@@ -193,7 +193,7 @@
           <mesh filename="package://ur_e_description/meshes/ur5e/visual/forearm.dae" />
         </geometry>
-        <material name="LightGrey">
-          <color rgba="0.7 0.7 0.7 1.0"/>
-        </material>
+        <!--material name="LightGrey">
+          <color rgba="0.7 0.7 0.7 1.0"/>
+        </material-->
       </visual>
       <collision>
@@ -230,7 +230,7 @@
           <mesh filename="package://ur_e_description/meshes/ur5e/visual/wrist1.dae" />
         </geometry>
-        <material name="LightGrey">
-          <color rgba="0.7 0.7 0.7 1.0"/>
-        </material>
+        <!--material name="LightGrey">
+          <color rgba="0.7 0.7 0.7 1.0"/>
+        </material-->
       </visual>
       <collision>
@@ -267,7 +267,7 @@
           <mesh filename="package://ur_e_description/meshes/ur5e/visual/wrist2.dae" />
         </geometry>
-        <material name="LightGrey">
-          <color rgba="0.7 0.7 0.7 1.0"/>
-        </material>
+        <!--material name="LightGrey">
+          <color rgba="0.7 0.7 0.7 1.0"/>
+        </material-->
       </visual>
       <collision>
@@ -304,7 +304,7 @@
           <mesh filename="package://ur_e_description/meshes/ur5e/visual/wrist3.dae" />
         </geometry>
-        <material name="LightGrey">
-          <color rgba="0.7 0.7 0.7 1.0"/>
-        </material>
+        <!--material name="LightGrey">
+          <color rgba="0.7 0.7 0.7 1.0"/>
+        </material-->
       </visual>
       <collision>
