Commit message: update for ur3e

File: ur_e_description/urdf/dual_ur3e_robot.urdf.xacro (robot description, xacro)
@@ -42,5 +42,5 @@
   <link name="dual_arm_base" >
     <visual>
-      <origin xyz="0 -0.4 0" rpy="1.5707963267949 0.0 0.0" />
+      <!--origin xyz="0 -0.4 0" rpy="1.5707963267949 0.0 0.0" /-->
       <geometry>
         <mesh filename="package://ur_e_description/meshes/ur5e/dual_ur5_base.stl" />
@@ -51,5 +51,5 @@
     </visual>
     <collision>
-      <origin xyz="0 -0.4 0" rpy="1.5707963267949 0.0 0.0" />
+      <!--origin xyz="0 -0.4 0" rpy="1.5707963267949 0.0 0.0" /-->
       <geometry>
         <mesh filename="package://ur_e_description/meshes/ur5e/dual_ur5_base.stl" />
@@ -150,5 +150,6 @@
     <origin xyz="0.0 0.0 0.52" rpy="0.0 0.0 0.0" />
   </joint>
-  <link name="dual_arm_booth">
+  <!-- booth -->
+  <!--link name="dual_arm_booth">
     <visual>
       <origin rpy="1.5707963267949 0.0 0.0" xyz="0 -0.75 0"/>
@@ -178,5 +179,5 @@
     <child link="dual_arm_booth"/>
     <origin rpy="0.0 0.0 0.0" xyz="-0.11 0.0 0.0"/>
-  </joint>
+  </joint-->
   <link name="display">
    <visual>

File: ur_e_description/urdf/ur3e.urdf.xacro (robot description, xacro)
@@ -56,5 +56,5 @@
     <!-- link lengths used in model -->
     <xacro:property name="shoulder_height" value="${d1}" />
-    <xacro:property name="upper_arm_length" value="${-a2}" />
+    <xacro:property name="upper_arm_length" value="${-a2 + 0.05555}" />
     <xacro:property name="forearm_length" value="${-a3}" />
     <xacro:property name="wrist_1_length" value="${d4}" />
